File: hardware/openRuche/open-ruche-monitoring.kicad_sch (KiCad schematic)
At the start: 20 parts, among them J1 HX711, J10 MMA8451, J11 CONN_LIPO, J12 CONN_ALIM_ESP32, J2 DHT22_EXT, J3 DHT22_INT, J4 SONDE_TEMP_1, J5 SONDE_TEMP_2, J6 Light Sensor, J7 LORA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

Commit message: hw(pcb) main pcb changes
Connections:
- net +3.3V: now also J7.2 (VCC)
- net +3.3V_REG: no longer J7.2 (VCC)
- net GND: now also U1.23 (GPIO18)
- no-connect marks 25 -> 24
Changed lines of the file:
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@@
-	)
-	(no_connect
-		(at 154.94 96.52)
 	)
 	(no_connect
@@
 	(wire
 		(pts
+			(xy 170.18 96.52) (xy 170.18 99.06)
+		)
+		(stroke
+			(width 0)
+			(type default)
+		)
+	)
+	(wire
+		(pts
 			(xy 144.78 185.42) (xy 147.32 185.42)
 		)
@@
 		(pts
 			(xy 241.3 36.83) (xy 251.46 36.83)
+		)
+		(stroke
+			(width 0)
+			(type default)
+		)
+	)
+	(wire
+		(pts
+			(xy 154.94 96.52) (xy 170.18 96.52)
 		)
 		(stroke
@@
 		)
 	)
-	(label "+3.3V_REG"
+	(label "+3.3V"
 		(at 93.98 185.42 180)
 		(effects
@@
 					(unit 1)
 				)
+			)
+		)
+	)
+	(symbol
+		(lib_id "power:GND")
+		(at 170.18 99.06 0)
+		(unit 1)
+		(exclude_from_sim no)
+		(in_bom yes)
+		(on_board yes)
+		(dnp no)
+		(fields_autoplaced yes)
+		(property "Reference" "#PWR012"
+			(at 170.18 105.41 0)
+			(effects
+				(font
+					(size 1.27 1.27)
+				)
+				(hide yes)
+			)
+		)
+		(property "Value" "GND"
+			(at 170.18 104.14 0)
+			(effects
+				(font
+					(size 1.27 1.27)
+				)
+			)
+		)
+		(property "Footprint" ""
+			(at 170.18 99.06 0)
+			(effects
+				(font
+					(size 1.27 1.27)
+				)
+				(hide yes)
+			)
+		)
+		(property "Datasheet" ""
+			(at 170.18 99.06 0)
+			(effects
+				(font
+					(size 1.27 1.27)
+				)
+				(hide yes)
+			)
+		)
+		(property "Description" "Power symbol creates a global label with name \"GND\" , ground"
+			(at 170.18 99.06 0)
+			(effects
+				(font
+					(size 1.27 1.27)
+				)
+				(hide yes)
+			)
+		)
+		(pin "1"
+		)
+		(instances
+			(project ""
+				(path "/e6969a1e-07e0-44a4-bb0c-208cafbc127d"
+					(reference "#PWR012")
+					(unit 1)
+				)
